Commit message: Successfull Pick and Drop

File: urdf/drone.urdf.xacro (robot description, xacro)
@@ -283,4 +283,108 @@
       velocity="1000000" />
   </joint>
+  <!-- Cylindrical Stand 1 -->
+  <link name="stand_1">
+    <visual>
+      <origin xyz="-0.007625 -0.007625 -0.01" rpy="0 0 0"/>
+      <geometry>
+        <cylinder radius="0.005" length="0.001"/>
+      </geometry>
+      <material name="WHITE_MTL"/>
+    </visual>
+    <collision>
+      <origin xyz="-0.007625 -0.007625 -0.01" rpy="0 0 0"/>
+      <geometry>
+        <cylinder radius="0.005" length="0.001"/>
+      </geometry>
+    </collision>
+    <inertial>
+      <mass value="0.001"/>
+      <origin xyz="0 0 0" rpy="0 0 0"/>
+      <inertia ixx="0.000000001" ixy="0" ixz="0" iyy="0.000000001" iyz="0" izz="0.000000001"/>
+    </inertial>
+  </link>
+  <joint name="stand_1_joint" type="fixed">
+    <parent link="base_link"/>
+    <child link="stand_1"/>
+    <origin xyz="-0.007625 -0.007625 -0.01" rpy="0 0 0"/>
+  </joint>
+  <!-- Cylindrical Stand 2 -->
+  <link name="stand_2">
+    <visual>
+      <origin xyz="-0.007625 0.007625 -0.01" rpy="0 0 0"/>
+      <geometry>
+        <cylinder radius="0.005" length="0.001"/>
+      </geometry>
+      <material name="WHITE_MTL"/>
+    </visual>
+    <collision>
+      <origin xyz="-0.007625 0.007625 -0.01" rpy="0 0 0"/>
+      <geometry>
+        <cylinder radius="0.005" length="0.001"/>
+      </geometry>
+    </collision>
+    <inertial>
+      <mass value="0.001"/>
+      <origin xyz="0 0 0" rpy="0 0 0"/>
+      <inertia ixx="0.000000001" ixy="0" ixz="0" iyy="0.000000001" iyz="0" izz="0.000000001"/>
+    </inertial>
+  </link>
+  <joint name="stand_2_joint" type="fixed">
+    <parent link="base_link"/>
+    <child link="stand_2"/>
+    <origin xyz="-0.007625 0.007625 -0.01" rpy="0 0 0"/>
+  </joint>
+  <!-- Cylindrical Stand 3 -->
+  <link name="stand_3">
+    <visual>
+      <origin xyz="0.007625 -0.007625 -0.01" rpy="0 0 0"/>
+      <geometry>
+        <cylinder radius="0.005" length="0.001"/>
+      </geometry>
+      <material name="WHITE_MTL"/>
+    </visual>
+    <collision>
+      <origin xyz="0.007625 -0.007625 -0.01" rpy="0 0 0"/>
+      <geometry>
+        <cylinder radius="0.005" length="0.001"/>
+      </geometry>
+    </collision>
+    <inertial>
+      <mass value="0.001"/>
+      <origin xyz="0 0 0" rpy="0 0 0"/>
+      <inertia ixx="0.000000001" ixy="0" ixz="0" iyy="0.000000001" iyz="0" izz="0.000000001"/>
+    </inertial>
+  </link>
+  <joint name="stand_3_joint" type="fixed">
+    <parent link="base_link"/>
+    <child link="stand_3"/>
+    <origin xyz="0.007625 -0.007625 -0.01" rpy="0 0 0"/>
+  </joint>
+  <!-- Cylindrical Stand 4 -->
+  <link name="stand_4">
+    <visual>
+      <origin xyz="0.007625 0.007625 -0.01" rpy="0 0 0"/>
+      <geometry>
+        <cylinder radius="0.005" length="0.001"/>
+      </geometry>
+      <material name="WHITE_MTL"/>
+    </visual>
+    <collision>
+      <origin xyz="0.007625 0.007625 -0.01" rpy="0 0 0"/>
+      <geometry>
+        <cylinder radius="0.005" length="0.001"/>
+      </geometry>
+    </collision>
+    <inertial>
+      <mass value="0.001"/>
+      <origin xyz="0 0 0" rpy="0 0 0"/>
+      <inertia ixx="0.000000001" ixy="0" ixz="0" iyy="0.000000001" iyz="0" izz="0.000000001"/>
+    </inertial>
+  </link>
+  <joint name="stand_4_joint" type="fixed">
+    <parent link="base_link"/>
+    <child link="stand_4"/>
+    <origin xyz="0.007625 0.007625 -0.01" rpy="0 0 0"/>
+  </joint>
 <!--
   <link name="imu_link">
@@ -378,3 +482,35 @@
     </plugin>
   </gazebo>
+  <!-- <gazebo reference="stand_1">
+      <sensor type="contact" name="stand_1_bumper">
+        <update_rate>10</update_rate>
+        <contact>
+          <collision>base_link_fixed_joint_lump__stand_1_collision</collision>
+        </contact>
+      </sensor>
+  </gazebo>
+  <gazebo reference="stand_2">
+      <sensor type="contact" name="stand_2_bumper">
+        <update_rate>10</update_rate>
+        <contact>
+          <collision>base_link_fixed_joint_lump__stand_2_collision_1</collision>
+        </contact>
+      </sensor>
+  </gazebo>
+  <gazebo reference="stand_3">
+      <sensor type="contact" name="stand_3_bumper">
+        <update_rate>10</update_rate>
+        <contact>
+          <collision>base_link_fixed_joint_lump__stand_3_collision_2</collision>
+        </contact>
+      </sensor>
+  </gazebo>
+  <gazebo reference="stand_4">
+      <sensor type="contact" name="stand_4_bumper">
+        <update_rate>10</update_rate>
+        <contact>
+          <collision>base_link_fixed_joint_lump__stand_4_collision_3</collision>
+        </contact>
+      </sensor>
+  </gazebo> -->
 </robot>

Commit message: Delivery Area Setup

File: urdf/drone.urdf.xacro (robot description, xacro)
@@ -387,4 +387,72 @@
     <origin xyz="0.007625 0.007625 -0.01" rpy="0 0 0"/>
   </joint>
+   <!-- Cylindrical Stand 4 -->
+  <link name="camera">
+    <visual>
+      <origin xyz="0.0 0.0 -0.005" rpy="0 0 0"/>
+      <geometry>
+        <box>
+          <size>0.005 0.005 0.005</size>
+        </box>
+      </geometry>
+      <material name="WHITE_MTL"/>
+    </visual>
+    <collision>
+      <origin xyz="0.0 0.0 -0.005" rpy="0 0 0"/>
+      <geometry>
+        <box>
+          <size>0.005 0.005 0.005</size>
+        </box>
+      </geometry>
+    </collision>
+    <inertial>
+      <mass value="0.001"/>
+      <origin xyz="0 0 0" rpy="0 0 0"/>
+      <inertia ixx="0.000000001" ixy="0" ixz="0" iyy="0.000000001" iyz="0" izz="0.000000001"/>
+    </inertial>
+  </link>
+  <joint name="camera_joint" type="fixed">
+    <parent link="base_link"/>
+    <child link="camera"/>
+    <origin xyz="0.0 0.0 -0.005" rpy="0 1.57 0"/>
+  </joint>
+  <gazebo reference="camera">
+    <sensor type="camera" name="bottom_camera_sensor">
+      <pose>0 0 0 0 0 0</pose>
+      <update_rate>30.0</update_rate>
+      <camera name="bottom_camera_sensor">
+        <horizontal_fov>1.3962634</horizontal_fov>
+        <image>
+          <width>800</width>
+          <height>800</height>
+          <format>R8G8B8</format>
+        </image>
+        <clip>
+          <near>0.02</near>
+          <far>300</far>
+        </clip>
+        <noise>
+          <type>gaussian</type>
+          <mean>0.0</mean>
+          <stddev>0.007</stddev>
+        </noise>
+      </camera>
+      <plugin name="bottom_camera_sensor_controller" filename="libgazebo_ros_camera.so">
+        <alwaysOn>true</alwaysOn>
+        <visualize>true</visualize>
+        <updateRate>0.0</updateRate>
+        <cameraName>/drone/bottom_camera_sensor</cameraName>
+        <imageTopicName>bottom_camera_sensor/image_raw</imageTopicName>
+        <cameraInfoTopicName>/drone/back_camera/bottom_camera_info</cameraInfoTopicName>
+        <frameName>bottom_camera_sensor</frameName>
+        <hackBaseline>0.07</hackBaseline>
+        <distortionK1>0.0</distortionK1>
+        <distortionK2>0.0</distortionK2>
+        <distortionK3>0.0</distortionK3>
+        <distortionT1>0.0</distortionT1>
+        <distortionT2>0.0</distortionT2>
+      </plugin>
+    </sensor>
+  </gazebo>
 <!--
   <link name="imu_link">
